File: kicad/mcu_board/mcu_board.kicad_pcb (KiCad board)
At the start: 2 copper layers, 61 parts, among them J1 Conn_01x01_Female, J10 Conn_01x01_Female, J11 Conn_01x01_Female, J12 Conn_01x01_Female, J13 Conn_01x01_Female, J14 Conn_01x01_Female, J15 Conn_01x01_Female, J16 Conn_01x01_Female, J17 Conn_01x01_Female, J18 Conn_01x01_Female, J19 Conn_01x01_Female, J2 Conn_01x06_Female, J20 Conn_01x01_Female, J21 Conn_01x01_Female, J22 Conn_01x01_Female, J23 Conn_01x01_Female, J24 Conn_01x01_Female, J25 Conn_01x01_Female, J26 Conn_01x01_Female, J27 Conn_01x01_Female, J3 Conn_01x01_Female, J4 Conn_01x01_Female, J5 Conn_01x01_Female, J6 Conn_01x01_Female, J7 Conn_01x01_Female, J8 Conn_01x01_Female, J9 Conn_01x01_Female, SW1 SW_Push, SW10 SW_Push, SW11 SW_Push, SW12 SW_Push, SW13 SW_Push, SW14 SW_Push, SW2 SW_Push, SW3 SW_Push, SW4 SW_Push, SW5 SW_Push, SW6 SW_Push, SW7 SW_Push, SW8 SW_Push, SW9 SW_Push, U1 ATmega32U4-AU, Y1 8MHz

Commit message: added 4 keys around USB connector
Parts:
- removed SW10 (x6), SW11, SW12, SW13, SW14: SW_Push, Button_Switch_Keyboard:SW_Cherry_MX1A_1.00u_Plate
- removed SW9: SW_Push, Button_Switch_Keyboard:SW_Cherry_MX1A_1.50u_Plate
- added C5: 22uF, Capacitor_Tantalum_SMD:CP_EIA-3216-18_Kemet-A, F.Cu at (75.5, 59.5)
- added D10: LED, LED_THT:LED_D3.0mm, F.Cu at (195.2, 68.1)
- added D11: LL4148, Diode_SMD:D_MiniMELF, F.Cu at (54.7, 53.0)
- added D12: LL4148, Diode_SMD:D_MiniMELF, F.Cu at (68.1, 50.3)
- added D13: LED, LED_THT:LED_D3.0mm, F.Cu at (80.3, 100.9)
- added D14: LED, LED_THT:LED_D3.0mm, F.Cu at (212.2, 87.1)
- added D15: LL4148, Diode_SMD:D_MiniMELF, F.Cu at (118.8, 3.38)
- added D16: LED, LED_THT:LED_D3.0mm, F.Cu at (99.3, 100.9)
- added D17: LL4148, Diode_SMD:D_MiniMELF, F.Cu at (118.8, 1.13)
- added D5: PRTR5V0U2X, Package_TO_SOT_SMD:SOT-143, F.Cu at (108.7, 28.2)
- added D6: LED, LED_THT:LED_D3.0mm, F.Cu at (198.2, 106.1)
- added D7: LED, LED_THT:LED_D3.0mm, F.Cu at (80.2, 81.9)
- added D8: LED, LED_THT:LED_D3.0mm, F.Cu at (99.2, 81.9)
- added D9: LED, LED_THT:LED_D3.0mm, F.Cu at (181.2, 87.1)
- added F1: 500mA, Fuse:Fuse_1206_3216Metric, F.Cu at (89.7, 43.1)
- added J28: Conn_01x01_Female, Connector_PinSocket_2.54mm:PinSocket_1x01_P2.54mm_Horizontal, F.Cu at (76.0, 47.4)
- added J29: Conn_01x01_Female, Connector_PinSocket_2.54mm:PinSocket_1x01_P2.54mm_Horizontal, F.Cu at (92.5, 28.2)
- added J30: Conn_01x01_Female, Connector_PinSocket_2.54mm:PinSocket_1x01_P2.54mm_Horizontal, F.Cu at (76.0, 43.8)
- added J31: Conn_01x01_Female, Connector_PinSocket_2.54mm:PinSocket_1x01_P2.54mm_Horizontal, F.Cu at (104.8, 19.8)
- added J32: Conn_01x01_Female, Connector_PinSocket_2.54mm:PinSocket_1x01_P2.54mm_Horizontal, F.Cu at (92.5, 35.4)
- added Q1: BC817, MMBTA42, Package_TO_SOT_SMD:SOT-23, F.Cu at (114.0, 19.8)
- added R4: 5.1k, Resistor_SMD:R_0603_1608Metric, F.Cu at (29.6, 62.0)
- added R5: 5.1k, Resistor_SMD:R_0603_1608Metric, F.Cu at (32.6, 62.0)
- added R6: 10k, Resistor_SMD:R_0603_1608Metric, F.Cu at (35.6, 62.0)
- added R7: 10R, Resistor_SMD:R_1210_3225Metric, F.Cu at (89.7, 45.9)
- added REF**: SW_Cherry_MX1A_1.00u_Plate, Button_Switch_Keyboard:SW_Cherry_MX1A_1.00u_Plate, F.Cu at (189.0, 39.0)
- added REF**: SW_Cherry_MX1A_1.00u_Plate, Button_Switch_Keyboard:SW_Cherry_MX1A_1.00u_Plate, F.Cu at (180.0, 58.0)
- added REF**: SW_Cherry_MX1A_1.00u_Plate, Button_Switch_Keyboard:SW_Cherry_MX1A_1.00u_Plate, F.Cu at (166.0, 77.0)
- added REF**: SW_Cherry_MX1A_1.00u_Plate, Button_Switch_Keyboard:SW_Cherry_MX1A_1.00u_Plate, F.Cu at (176.0, 96.0)
- added REF**: SW_Cherry_MX1A_1.00u_Plate, Button_Switch_Keyboard:SW_Cherry_MX1A_1.00u_Plate, F.Cu at (228.0, 96.0)
- added REF**: SW_Cherry_MX1A_1.50u_Plate, Button_Switch_Keyboard:SW_Cherry_MX1A_1.50u_Plate, F.Cu at (223.0, 58.0)
- U1, USB1: moved to B.Cu
- moved SW5 180.4 mm to (79.0, 111.0), turned to 180 degrees
- moved SW7 154.1 mm to (98.0, 92.0), turned to 180 degrees
- moved C1 126.0 mm to (17.5, 62.0)
- moved C3 123.6 mm to (14.5, 62.0)
- moved R2 120.8 mm to (23.5, 62.0)
- moved C2 117.9 mm to (11.5, 62.0)
- moved SW6 117.6 mm to (98.0, 111.0), turned to 180 degrees
- moved R3 117.6 mm to (26.6, 62.0)
- moved C4 112.0 mm to (20.5, 62.0)
- moved J15 106.2 mm to (32.9, 59.4)
- moved D4 104.7 mm to (118.8, 5.63)
- moved D2 102.2 mm to (118.8, 7.88)
- moved SW8 102.2 mm to (79.0, 92.0), turned to 180 degrees
- moved J9 94.9 mm to (102.0, 9.03)
- moved J1 94.7 mm to (20.6, 59.4)
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Connections:
- net Net-(D3-Pad1) renamed /row_4
- net Net-(J1-Pad1) renamed /row_0
- net Net-(J2-Pad5) renamed /row_1
- net Net-(J5-Pad1) renamed /backlight
- D1 pad 1: Net-(D1-Pad1) -> /row_3
- D2 pad 1: Net-(D2-Pad1) -> /row_2
- D4 pad 1: Net-(D4-Pad1) -> /row_3
- J2 pad 3: Net-(J2-Pad3) -> /row_2
- J2 pad 4: Net-(J2-Pad4) -> /row_3
- J20 pad 1: Net-(J20-Pad1) -> /col_12
- J21 pad 1: Net-(J21-Pad1) -> /col_13
- J26 pad 1: Net-(J2-Pad3) -> /row_2
- J27 pad 1: Net-(J2-Pad4) -> /row_3
- J7 pad 1: Net-(J7-Pad1) -> /col_1
- J8 pad 1: Net-(J8-Pad1) -> /col_2
- SW1 pad 2: Net-(SW1-Pad2) -> /col_13
- SW2 pad 1: Net-(SW2-Pad1) -> Net-(D3-Pad2)
- SW2 pad 2: Net-(D3-Pad2) -> /col_13
- SW3 pad 1: Net-(SW3-Pad1) -> Net-(D4-Pad2)
- SW3 pad 2: Net-(D4-Pad2) -> /col_13
- SW4 pad 1: Net-(SW4-Pad1) -> Net-(D1-Pad2)
- SW4 pad 2: Net-(D1-Pad2) -> /col_12
- SW5 pad 2: Net-(SW5-Pad2) -> /col_1
- SW6 pad 2: Net-(SW6-Pad2) -> /col_2
- SW7 pad 2: Net-(SW7-Pad2) -> /col_1
- SW8 pad 2: Net-(SW8-Pad2) -> /col_2
- U1 pad 10: Net-(J2-Pad3) -> /row_2
- U1 pad 11: Net-(J2-Pad4) -> /row_3
- U1 pad 31: Net-(J7-Pad1) -> /col_1
- U1 pad 32: Net-(J8-Pad1) -> /col_2
- U1 pad 39: Net-(J21-Pad1) -> /col_13
- U1 pad 40: Net-(J20-Pad1) -> /col_12
- USB1 pad 11: +5V -> Net-(C5-Pad1)
- USB1 pad 2: +5V -> Net-(C5-Pad1)

Commit message: some pcb arrangement
Parts:
- added J33: Conn_01x01_Female, Connector_Wire:SolderWirePad_1x01_Drill0.8mm, F.Cu at (113.7, 91.4)
- added J34: Conn_01x01_Female, Connector_Wire:SolderWirePad_1x01_Drill0.8mm, F.Cu at (113.7, 94.6)
- added J35: Conn_01x01_Female, Connector_Wire:SolderWirePad_1x01_Drill0.8mm, F.Cu at (113.7, 101.0)
- added J36: Conn_01x01_Female, Connector_Wire:SolderWirePad_1x01_Drill0.8mm, F.Cu at (158.8, 104.8)
- added J37: Conn_01x01_Female, Connector_Wire:SolderWirePad_1x01_Drill0.8mm, F.Cu at (113.7, 97.8)
- added J38: Conn_01x01_Female, Connector_Wire:SolderWirePad_1x01_Drill0.8mm, F.Cu at (158.8, 98.4)
- added J39: Conn_01x01_Female, Connector_Wire:SolderWirePad_1x01_Drill0.8mm, F.Cu at (158.8, 95.2)
- added J40: Conn_01x01_Female, Connector_Wire:SolderWirePad_1x01_Drill0.8mm, F.Cu at (188.0, 132.7)
- added J41: Conn_01x01_Female, Connector_Wire:SolderWirePad_1x01_Drill0.8mm, F.Cu at (151.8, 71.1)
- added J42: Conn_01x01_Female, Connector_Wire:SolderWirePad_1x01_Drill0.8mm, F.Cu at (174.6, 144.8)
- added J43: Conn_01x01_Female, Connector_Wire:SolderWirePad_1x01_Drill0.8mm, F.Cu at (224.2, 126.4)
- added J44: Conn_01x01_Female, Connector_Wire:SolderWirePad_1x01_Drill0.8mm, F.Cu at (157.5, 139.1)
- added J45: Conn_01x01_Female, Connector_Wire:SolderWirePad_1x01_Drill0.8mm, F.Cu at (161.3, 120.7)
- added J46: Conn_01x01_Female, Connector_Wire:SolderWirePad_1x01_Drill0.8mm, F.Cu at (113.7, 109.9)
- added J47: Conn_01x01_Female, Connector_Wire:SolderWirePad_1x01_Drill0.8mm, F.Cu at (67.3, 83.8)
- added J48: Conn_01x01_Female, Connector_Wire:SolderWirePad_1x01_Drill0.8mm, F.Cu at (158.8, 101.6)
- added REF**: SW_Cherry_MX1A_1.00u_Plate, Button_Switch_Keyboard:SW_Cherry_MX1A_1.00u_Plate, F.Cu at (190.0, 115.0)
- added REF**: SW_Cherry_MX1A_1.00u_Plate, Button_Switch_Keyboard:SW_Cherry_MX1A_1.00u_Plate, F.Cu at (228.0, 115.0)
- added REF**: SW_Cherry_MX1A_1.00u_Plate, Button_Switch_Keyboard:SW_Cherry_MX1A_1.00u_Plate, F.Cu at (209.0, 115.0)
- C1, C2, C3, C4, C5, D1, D11, D12, D15, D17, D2, D3, D4, D5, F1, Q1, R1, R2, R3, R4, R5, R6, R7, Y1: moved to B.Cu
- J1, J10, J11, J12, J13, J14, J15, J16, J17, J18, J19, J20, J21, J22, J23, J24, J25, J26, J27, J28, J29, J3, J30, J31, J32, J4, J5, J6, J7, J8, J9: footprint Connector_PinSocket_2.54mm:PinSocket_1x01_P2.54mm_Horizontal -> Connector_Wire:SolderWirePad_1x01_Drill0.8mm
- moved J1 214.7 mm to (234.9, 70.5)
- moved J3 206.7 mm to (251.0, 79.0)
- moved J15 202.9 mm to (235.0, 78.0)
- moved C2 186.8 mm to (198.0, 72.0)
- moved C1 185.9 mm to (203.0, 75.0), turned to 90 degrees
- moved J7 180.4 mm to (235.0, 93.0)
- moved C4 177.2 mm to (194.8, 94.0), turned to 180 degrees
- moved J2 177.0 mm to (223.5, 76.2)
- moved J26 175.0 mm to (244.0, 82.0)
- moved C3 173.4 mm to (186.7, 82.3), turned to 270 degrees
- moved R6 173.2 mm to (208.3, 74.8), turned to 270 degrees
- moved J5 170.8 mm to (249.0, 93.0)
- moved J24 170.1 mm to (218.0, 117.0)
- moved R3 167.6 mm to (193.5, 76.2)
- moved R2 167.3 mm to (189.1, 86.4), turned to 180 degrees
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Connections:
- net Net-(C5-Pad1) renamed /VBUS
- J25 pad 1: /row_1 -> /row_4
- R1 pad 1: /D- -> Net-(R1-Pad1)
- R1 pad 2: Net-(R1-Pad2) -> /D+
- R2 pad 1: /D+ -> Net-(R2-Pad1)
- R2 pad 2: Net-(R2-Pad2) -> /D-
- R4 pad 1: Net-(R2-Pad2) -> /D-
- R5 pad 1: Net-(R1-Pad2) -> /D+
- U1 pad 3: /D- -> Net-(R2-Pad1)
- U1 pad 4: /D+ -> Net-(R1-Pad1)
- USB1 pad 5: Net-(R1-Pad2) -> /D-
- USB1 pad 6: Net-(R2-Pad2) -> /D+
- USB1 pad 7: Net-(R1-Pad2) -> /D-
- USB1 pad 8: Net-(R2-Pad2) -> /D+

Commit message: pcb
Parts:
- removed REF** (x8): SW_Cherry_MX1A_1.00u_Plate, Button_Switch_Keyboard:SW_Cherry_MX1A_1.00u_Plate
- removed REF**: SW_Cherry_MX1A_1.50u_Plate, Button_Switch_Keyboard:SW_Cherry_MX1A_1.50u_Plate
- removed REF**: SW_Cherry_MX1A_2.00u_Plate, Button_Switch_Keyboard:SW_Cherry_MX1A_2.00u_Plate
- added J49: Conn_01x01_Female, Connector_Wire:SolderWirePad_1x01_Drill0.8mm, F.Cu at (144.5, 91.5)
- added J50: Conn_01x01_Female, Connector_Wire:SolderWirePad_1x01_Drill0.8mm, F.Cu at (163.5, 91.5)
- added J51: Conn_01x01_Female, Connector_Wire:SolderWirePad_1x01_Drill0.8mm, F.Cu at (153.5, 91.5)
- added J52: Conn_01x01_Female, Connector_Wire:SolderWirePad_1x01_Drill0.8mm, F.Cu at (204.0, 55.0)
- J2: moved to B.Cu
- moved J42 95.8 mm to (208.0, 55.0)
- moved J44 91.7 mm to (194.0, 55.0)
- moved J31 91.1 mm to (170.0, 88.5)
- moved SW8 83.2 mm to (159.5, 71.0)
- moved J5 78.3 mm to (174.0, 70.5)
- moved J3 77.2 mm to (174.0, 73.5)
- moved J40 74.7 mm to (187.5, 58.0)
- moved J30 72.4 mm to (135.0, 82.5)
- moved J8 71.0 mm to (170.0, 91.5)
- moved J45 70.7 mm to (187.5, 55.0)
- moved J47 70.3 mm to (135.0, 65.0)
- moved J46 68.7 mm to (170.0, 70.5)
- moved J12 66.3 mm to (187.5, 106.5)
- moved D11 66.3 mm to (139.0, 84.2)
- moved D13 65.0 mm to (141.8, 79.9)
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Connections:
- net Net-(J10-Pad1) renamed /col_4
- net Net-(J11-Pad1) renamed /col_5
- net Net-(J12-Pad1) renamed /col_6
- net Net-(J13-Pad1) renamed /col_7
- net Net-(J14-Pad1) renamed /col_8
- net Net-(J15-Pad1) renamed /col_9
- net Net-(J16-Pad1) renamed /col_10
- net Net-(J17-Pad1) renamed /unused_1
- net Net-(J18-Pad1) renamed /unused_2
- net Net-(J19-Pad1) renamed /col_11
- net Net-(J22-Pad1) renamed /col_14
- net Net-(J23-Pad1) renamed /col_15
- net Net-(J24-Pad1) renamed /unused_3
- net Net-(J4-Pad1) renamed /row_5
- net Net-(J6-Pad1) renamed /col_0
- net Net-(J9-Pad1) renamed /col_3
- J3 pad 1: Net-(J3-Pad1) -> /BL_cathode
- J42 pad 1: /col_13 -> /BL_cathode
- J5 pad 1: /backlight -> /row_1
- U1 pad 28: Net-(J3-Pad1) -> /row_4
Routing:
- net /BL_cathode: track 0.00 -> 97.7 mm, vias 0 -> 4
- net /col_1: track 0.00 -> 81.2 mm, vias 0 -> 3
- net /row_1: track 0.00 -> 49.3 mm, vias 0 -> 1
- net /row_0: track 0.00 -> 48.0 mm, vias 0 -> 1
- net /VBUS: track 0.00 -> 47.8 mm, vias 0 -> 2
- net /D-: track 0.00 -> 45.8 mm, vias 0 -> 2
- net /D+: track 0.00 -> 44.3 mm, vias 0 -> 2
- net /col_2: track 0.00 -> 30.6 mm, vias 0 -> 1
- net +5V: track 0.00 -> 30.2 mm, vias 0 -> 2
- net Net-(D17-Pad2): track 0.00 -> 23.2 mm
- net Net-(D15-Pad2): track 0.00 -> 20.3 mm
- net /col_12: track 0.00 -> 15.6 mm
- net /row_3: track 0.00 -> 14.0 mm
- net /col_13: track 0.00 -> 8.85 mm
- net GND: track 0.00 -> 7.74 mm
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- added copper zone on F.Cu, net +5V
- added copper zone on B.Cu, net GND
Other:
- board outline added: 92 x 54.5 mm
- net class power added: clearance 0.2, trace_width 0.4, via_dia 0.8, via_drill 0.4

Commit message: pcb
Parts:
- moved C4 17.0 mm to (207.5, 81.7)
- moved C1 14.2 mm to (194.3, 90.3), turned to 270 degrees
- moved J4 13.1 mm to (192.4, 106.5)
- moved J21 12.6 mm to (206.1, 106.5)
- moved R4 12.2 mm to (209.5, 71.0)
- moved SW1 11.4 mm to (193.5, 68.0), turned to 180 degrees
- moved SW2 11.4 mm to (196.5, 106.0), turned to 180 degrees
- moved SW4 11.4 mm to (179.5, 87.0), turned to 180 degrees
- moved SW3 11.4 mm to (210.5, 87.0), turned to 180 degrees
- moved D10 10.2 mm to (194.8, 57.9)
- moved D14 10.2 mm to (211.8, 76.9)
- moved D6 10.2 mm to (197.8, 95.9)
- moved D9 10.2 mm to (180.8, 76.9)
- moved J12 9.00 mm to (187.5, 97.5)
- moved J9 9.00 mm to (187.5, 106.5)
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Routing:
- net GND: track 7.74 -> 112.4 mm, vias 0 -> 9
- net /BL_cathode: track 97.7 -> 199.3 mm, vias 4 -> 9
- net /row_2: track 0.00 -> 87.0 mm, vias 0 -> 7
- net +5V: track 30.2 -> 115.1 mm, vias 2 -> 13
- net /col_13: track 8.85 -> 86.4 mm, vias 0 -> 4
- net /row_1: track 49.3 -> 113.2 mm, vias 1 -> 10
- net /row_3: track 14.0 -> 71.0 mm, vias 0 -> 5
- net /D+: track 44.3 -> 96.4 mm, vias 2 -> 7
- net /row_4: track 0.00 -> 49.1 mm, vias 0 -> 2
- net /D-: track 45.8 -> 89.4 mm, vias 2 -> 8
- net /unused_1: track 0.00 -> 42.8 mm, vias 0 -> 2
- net /col_2: track 30.6 -> 70.1 mm, vias 1 -> 4
- net /unused_2: track 0.00 -> 38.9 mm, vias 0 -> 2
- net /row_0: track 48.0 -> 86.8 mm, vias 1 -> 5
- net /col_12: track 15.6 -> 53.9 mm, vias 0 -> 3
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
Commit message: pcb
Other:
- board text added: "+5v"
- board text added: "BL"
- board text added: "D+"
- board text added: "D-"
- board text added: "GND"
- board text added: "VBUS"
- board text added: "c0"
- board text added: "c1"
- board text added: "c10"
- board text added: "c11"
- board text added: "c12"
- board text added: "c13"
- board text added: "c14"
- board text added: "c15"
- board text added: "c2"
- board text added: "c3"
- board text added: "c4"
- board text added: "c5"
- board text added: "c6"
- board text added: "c7"
- board text added: "c8"
- board text added: "c9"
- board text added: "prog"
- board text added: "r0"
- board text added: "r1"
- board text added: "r2"
- board text added: "r3"
- board text added: "r4"
- board text added: "r5"
- board text added: "u1"
- board text added: "u2"
- board text added: "u3"
